File: LEVIA_H7.kicad_pcb (KiCad board)
At the start: 6 copper layers, 39.5 x 39.5 mm, 168 parts, among them J1 TF-028-H265, Q1 AO3400A, SW2 RKCGG140SMTRLFS, U1 USBLC6-2P6, U10 ZX-SH1.0-4PWT, U11 ZX-SH1.0-3PWT, U12 SIT1051TK/3, U13 ZX-SH1.0-4PWT, U14 ICM-42688-P, U15 ICM-42688-P, U16 DPS368XTSA1, U17 IST8310, U18 ZX-SH1.0-4PWT, U19 ZX-SH1.0-6PWT, U2 STM32H743VIHx, U20 ZX-SH1.0-6PWT, U21 ZX-SH1.0-3PWT, U22 ZX-SH1.0-8PWT, U24 ZX-SH1.0-4PWT, U3 ZX-SH1.0-4PWT, U4 LMR43620R5RPER, U5 LMR604303SRAKRQ1, U6 AP7361C-33FGE-7, U7 AP7361C-33FGE-7, U8 ZX-SH1.0-4PWT, U9 AT7456ELAH, Y1 8MHz, Y2 XL7EL89COI-111YLC-27M

Commit message: DFA2 gerbers
Parts:
- added H1: MountingHole_Pad, _pico:MountingHole_3.2mm_M3_ISO14580_Pad_TopBottom, F.Cu at (154.0, 53.8)
- added H2: MountingHole_Pad, _pico:MountingHole_3.2mm_M3_ISO14580_Pad_TopBottom, F.Cu at (154.0, 84.4)
- added H3: MountingHole_Pad, _pico:MountingHole_3.2mm_M3_ISO14580_Pad_TopBottom, F.Cu at (123.5, 84.4)
- added H4: MountingHole_Pad, _pico:MountingHole_3.2mm_M3_ISO14580_Pad_TopBottom, F.Cu at (123.5, 53.9)
- added REF**: OSHW-Logo2_7.3x6mm_SilkScreen, Symbol:OSHW-Logo2_7.3x6mm_SilkScreen, F.Cu at (143.9, 60.6)
